File: PCB/Virgil Controller/Power.kicad_sch (KiCad schematic)
At the start: 8 parts, among them J2 Conn_02x25_Odd_Even, U28 SN74CBTLV1G125DCKR

Commit message: Created actually good readme
Parts:
- removed TP1, TP2: B+, TestPoint:TestPoint_Pad_D4.0mm, symbol Connector:TestPoint
- removed TP3: M1, TestPoint:TestPoint_Pad_D2.0mm, symbol Connector:TestPoint
- removed TP4: M0, TestPoint:TestPoint_Pad_D2.0mm, symbol Connector:TestPoint
- removed TP5: M3, TestPoint:TestPoint_Pad_D2.0mm, symbol Connector:TestPoint
- removed TP6: M2, TestPoint:TestPoint_Pad_D2.0mm, symbol Connector:TestPoint
Connections:
- removed net B+: J2.10 (Pin_10), J2.11 (Pin_11), J2.12 (Pin_12), J2.9 (Pin_9)
- removed net B-: J2.1 (Pin_1), J2.2 (Pin_2), J2.3 (Pin_3), J2.4 (Pin_4)
- net M0: no longer names the net of J2.6 (Pin_6)
- net M1: no longer names the net of J2.5 (Pin_5)
- net M2: no longer names the net of J2.8 (Pin_8)
- net M3: no longer names the net of J2.7 (Pin_7)
- no-connect marks 0 -> 12
