File: PCB/Virgil Controller/Networking.kicad_sch (KiCad schematic)
At the start: 14 parts, among them J19 NE8FAH, T2 PT61018PEL, U12 W5500IO, U5 SC1169

Commit message: Created actually good readme
Parts:
- removed U12: W5500IO, Snapeda:W5500-io, symbol Snapeda:W5500io
- added C16: 4.7uF, Capacitor_SMD:C_0805_2012Metric, symbol Device:C
- added C17, C18: .1uF, Capacitor_SMD:C_0603_1608Metric, symbol Device:C
- added C19: 22nF, Capacitor_SMD:C_0603_1608Metric, symbol Device:C
- added C20, C21: 18pF, Capacitor_SMD:C_0603_1608Metric, symbol Device:C
- added D13, D14: LED, LED_SMD:LED_0603_1608Metric, symbol Device:LED
- added R10: 12.4kΩ, Resistor_SMD:R_0603_1608Metric, symbol Device:R_US
- added R11, R12, R13, R14: 3.3Ω, Resistor_SMD:R_0603_1608Metric, symbol Device:R_US
- added R15, R16, R17, R18: 49.9kΩ, Resistor_SMD:R_0603_1608Metric, symbol Device:R_US
- added R19: 10Ω, Resistor_SMD:R_0603_1608Metric, symbol Device:R_US
- added R7, R8: 68Ω, Resistor_SMD:R_0603_1608Metric, symbol Device:R_US
- added R9: 1MΩ, Resistor_SMD:R_0603_1608Metric, symbol Device:R_US
- added TP17: DUPLED, Connector_PinHeader_2.00mm:PinHeader_1x01_P2.00mm_Vertical, symbol Connector:TestPoint
- added TP18: ACTLED, Connector_PinHeader_2.00mm:PinHeader_1x01_P2.00mm_Vertical, symbol Connector:TestPoint
- added U4: W5500, Package_QFP:LQFP-48_7x7mm_P0.5mm, symbol Interface_Ethernet:W5500
- added Y2: 25MHZ, Crystal:Crystal_SMD_Abracon_ABM3C-4Pin_5.0x3.2mm, symbol Device:Crystal_GND24
- TP15: value DUPLED -> SPDLED
- TP16: value ACTLED -> LINKLED
Connections:
- net +3.3V: now also R15.1, R16.1, R19.1, R7.1, R8.1, U4.11 (AVDD), U4.15 (AVDD), U4.17 (AVDD), U4.21 (AVDD), U4.28 (VDD), U4.4 (AVDD), U4.43 (PMODE2), U4.44 (PMODE1), U4.45 (PMODE0), U4.8 (AVDD)
- net CLK: now also U4.33 (SCLK)
- net GND: now also C16.1, C17.1, C18.1, C19.2, C20.2, C21.2, R10.2, U4.14 (AGND), U4.16 (AGND), U4.19 (AGND), U4.29 (GND), U4.3 (AGND), U4.48 (AGND), U4.9 (AGND), Y2.2 (G), Y2.4 (G)
- net MISO: now also U4.34 (MISO)
- net MOSI: now also U4.35 (MOSI)
- net RX+: now also R14.2, R18.2
- net RX-: now also R13.2, R17.2
- net TX+: now also R12.2, R16.2
- net TX-: now also R11.2, R15.2
- net W5500_~{CS}: now also U4.32 (~{SCS})
- net W5500_~{INT}: now also U4.36 (~{INT})
- net W5500_~{RESET}: now also U4.37 (~{RST})
- net TCT: now reaches T2.2 (CT1)
- net TCT: now also C19.1, R19.2
- net RCT: now reaches T2.7 (CT2)
- net RCT: now also C18.2, R17.1, R18.1
- net at D12.2 (A), TP16.1: now also U4.25 (LINKLED)
- net at D11.2 (A), TP15.1: now also U4.24 (SPDLED)
- new net: D14.1 (K), R8.2
- new net: C20.1, R9.1, U4.30 (XI/CLKIN), Y2.1
- new net: C21.1, R9.2, U4.31 (XO), Y2.3
- new net: R14.1, U4.6 (RXP)
- new net: R11.1, U4.1 (TXN)
- new net: R12.1, U4.2 (TXP)
- new net: D14.2 (A), TP18.1, U4.27 (ACTLED)
- new net: R13.1, U4.5 (RXN)
- new net: D13.2 (A), TP17.1, U4.26 (DUPLED)
- new net: C16.2, U4.20 (TOCAP)
- new net: D13.1 (K), R7.2
- new net: C17.2, U4.22 (1V2O)
- new net: R10.1, U4.10 (EXRES1)
- no-connect marks 0 -> 7
Other:
- moved on the sheet: D11, D12, R3, R6, TP15, TP16

Commit message: Finished PCBs
Parts:
- Y2: value 25MHZ -> ABM3C-25.000MHZ-D4Y-T
Changed lines of the file:
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@@
 			)
 		)
-		(property "Value" "25MHZ"
+		(property "Value" "ABM3C-25.000MHZ-D4Y-T"
 			(at 112.395 104.14 0)
 			(show_name no)
