File: PCB/Virgil Controller/Virgil Controller.kicad_pcb (KiCad board)
At the start: 2 copper layers, 128.1 x 87 mm, 34 parts, among them J1 USB_C_Receptacle_USB2.0_16P, J19 NE8FAH, J2 Conn_02x25_Odd_Even, J3 503398-1892, J6 SBH11-PBPC-D25-RA-BK, T2 PT61018PEL, U12 W5500IO, U28 SN74CBTLV1G125DCKR, U4 RP2350_Stamp_XL, U5 SC1169

Commit message: Created actually good readme
Parts:
- removed TP1, TP2: B+, TestPoint:TestPoint_Pad_D4.0mm
- removed TP3: M1, TestPoint:TestPoint_Pad_D2.0mm
- removed TP4: M0, TestPoint:TestPoint_Pad_D2.0mm
- removed TP5: M3, TestPoint:TestPoint_Pad_D2.0mm
- removed TP6: M2, TestPoint:TestPoint_Pad_D2.0mm
- removed TP77: BootSel, Connector_PinHeader_2.00mm:PinHeader_1x01_P2.00mm_Vertical
- removed U12: W5500IO, Snapeda:W5500-io
- added C1: 4.7uF, Capacitor_SMD:C_0805_2012Metric, F.Cu at (198.0, 128.9)
- added C10: .1uF, Capacitor_SMD:C_0603_1608Metric, F.Cu at (185.3, 135.2)
- added C11: .1uF, Capacitor_SMD:C_0603_1608Metric, F.Cu at (205.2, 141.6)
- added C12: .1uF, Capacitor_SMD:C_0603_1608Metric, F.Cu at (187.7, 145.5)
- added C13: 4.7uF, Capacitor_SMD:C_0805_2012Metric, F.Cu at (187.9, 125.0)
- added C14: 22pF, Capacitor_SMD:C_0603_1608Metric, F.Cu at (206.8, 147.3)
- added C15: 22pF, Capacitor_SMD:C_0603_1608Metric, F.Cu at (207.3, 143.0)
- added C16: 4.7uF, Capacitor_SMD:C_0805_2012Metric, F.Cu at (141.4, 136.9)
- added C17: .1uF, Capacitor_SMD:C_0603_1608Metric, F.Cu at (141.6, 138.8)
- added C18: .1uF, Capacitor_SMD:C_0603_1608Metric, F.Cu at (155.9, 125.6)
- added C19: 22nF, Capacitor_SMD:C_0603_1608Metric, F.Cu at (146.6, 125.6)
- added C2: .1uF, Capacitor_SMD:C_0603_1608Metric, F.Cu at (188.6, 132.2)
- added C20: 18pF, Capacitor_SMD:C_0603_1608Metric, F.Cu at (146.4, 146.2)
- added C21: 18pF, Capacitor_SMD:C_0603_1608Metric, F.Cu at (154.2, 146.3)
- added C3: .1uF, Capacitor_SMD:C_0603_1608Metric, F.Cu at (193.3, 130.8)
- added C4: .1uF, Capacitor_SMD:C_0603_1608Metric, F.Cu at (202.1, 132.1)
- added C5: .1uF, Capacitor_SMD:C_0603_1608Metric, F.Cu at (201.8, 146.0)
- added C6: .1uF, Capacitor_SMD:C_0603_1608Metric, F.Cu at (198.6, 147.3)
- added C7: .1uF, Capacitor_SMD:C_0603_1608Metric, F.Cu at (203.9, 136.1)
- added C8: .1uF, Capacitor_SMD:C_0603_1608Metric, F.Cu at (185.2, 143.2)
- added C9: .1uF, Capacitor_SMD:C_0603_1608Metric, F.Cu at (190.0, 147.9)
- added D13: LED, LED_SMD:LED_0603_1608Metric, F.Cu at (140.8, 149.1)
- added D14: LED, LED_SMD:LED_0603_1608Metric, F.Cu at (143.9, 149.2)
- added J4: Conn_01x03_Pin, Connector_PinSocket_2.54mm:PinSocket_1x03_P2.54mm_Vertical, F.Cu at (229.3, 130.7)
- added L1: 3.3uH, Inductor_SMD:L_Pulse_PA4340, F.Cu at (191.9, 126.8)
- added R10: 12.4kΩ, Resistor_SMD:R_0603_1608Metric, F.Cu at (147.4, 129.4)
- added R11: 3.3Ω, Resistor_SMD:R_0603_1608Metric, F.Cu at (149.7, 125.6)
- added R12: 3.3Ω, Resistor_SMD:R_0603_1608Metric, F.Cu at (143.5, 125.6)
- added R13: 3.3Ω, Resistor_SMD:R_0603_1608Metric, F.Cu at (158.3, 124.8)
- added R14: 3.3Ω, Resistor_SMD:R_0603_1608Metric, F.Cu at (152.8, 125.6)
- added R15: 49.9kΩ, Resistor_SMD:R_0603_1608Metric, F.Cu at (149.7, 124.0)
- added R16: 49.9kΩ, Resistor_SMD:R_0603_1608Metric, F.Cu at (143.5, 124.0)
- added R17: 49.9kΩ, Resistor_SMD:R_0603_1608Metric, F.Cu at (155.9, 124.0)
- added R18: 49.9kΩ, Resistor_SMD:R_0603_1608Metric, F.Cu at (152.8, 124.0)
- added R19: 10Ω, Resistor_SMD:R_0603_1608Metric, F.Cu at (146.6, 124.0)
- added R20: 27Ω, Resistor_SMD:R_0603_1608Metric, F.Cu at (186.8, 127.7)
- added R21: 27Ω, Resistor_SMD:R_0603_1608Metric, F.Cu at (185.7, 128.8)
- added R4: 4.7Ω, Resistor_SMD:R_0805_2012Metric, F.Cu at (218.9, 157.0)
- added R5: 4.7Ω, Resistor_SMD:R_0805_2012Metric, F.Cu at (218.9, 154.8)
- added R7: 68Ω, Resistor_SMD:R_0603_1608Metric, F.Cu at (140.8, 152.5)
- added R8: 68Ω, Resistor_SMD:R_0603_1608Metric, F.Cu at (143.9, 152.5)
- added R9: 1MΩ, Resistor_SMD:R_0603_1608Metric, F.Cu at (149.0, 148.7)
- added TP17: DUPLED, Connector_PinHeader_2.00mm:PinHeader_1x01_P2.00mm_Vertical, F.Cu at (140.8, 145.9)
- added TP18: ACTLED, Connector_PinHeader_2.00mm:PinHeader_1x01_P2.00mm_Vertical, F.Cu at (143.9, 145.9)
- added U1: RP2350B, Package_DFN_QFN:QFN-80-1EP_10x10mm_P0.4mm_EP3.4x3.4mm, F.Cu at (194.9, 138.9)
- added U2: W25Q16JVSS, Package_SO:SOIC-8_5.3x5.3mm_P1.27mm, F.Cu at (179.1, 131.5)
- added U3: W25Q16JVSS, Package_SO:SOIC-8_5.3x5.3mm_P1.27mm, F.Cu at (174.9, 127.0)
- added Y1: Crystal_GND24, Crystal:Crystal_SMD_Abracon_ABM8G-4Pin_3.2x2.5mm, F.Cu at (205.2, 145.2)
- added Y2: 25MHZ, Crystal:Crystal_SMD_Abracon_ABM3C-4Pin_5.0x3.2mm, F.Cu at (150.3, 145.7)
- R1: value 4.7Ω -> 33Ω; footprint Resistor_SMD:R_0805_2012Metric -> Resistor_SMD:R_0603_1608Metric
- R2: value 4.7Ω -> 1kΩ; footprint Resistor_SMD:R_0805_2012Metric -> Resistor_SMD:R_0603_1608Metric
- TP15: value DUPLED -> SPDLED
- TP16: value ACTLED -> LINKLED
- U4: value RP2350_Stamp_XL -> W5500; footprint Snapeda:RP2xxx_Stamp_XL_FlexyPin -> Package_QFP:LQFP-48_7x7mm_P0.5mm
- moved TP78 55.7 mm to (229.3, 120.5), turned to 0 degrees
- moved U4 40.1 mm to (150.0, 136.1), turned to -90 degrees
- moved R1 34.9 mm to (196.5, 130.3), turned to 135 degrees
- moved R2 19.3 mm to (203.0, 143.8), turned to 45 degrees
- moved TP16 15.2 mm to (137.7, 145.9), turned to 0 degrees
- moved D12 12.4 mm to (137.7, 149.1)
- moved R6 10.7 mm to (137.7, 152.5), turned to 90 degrees
- moved T2 8.73 mm to (151.1, 116.0)
- moved TP15 6.24 mm to (134.6, 145.9), turned to 0 degrees
- moved U28 5.11 mm to (120.0, 129.0)
- moved R3 1.98 mm to (134.6, 152.5)
- moved D11 1.96 mm to (134.6, 149.1), turned to 90 degrees
Connections:
- J2 pad 1: /Power/B- -> unconnected-(J2-Pin_1-Pad1)
- J2 pad 10: /Power/B+ -> unconnected-(J2-Pin_10-Pad10)
- J2 pad 11: /Power/B+ -> unconnected-(J2-Pin_11-Pad11)
- J2 pad 12: /Power/B+ -> unconnected-(J2-Pin_12-Pad12)
- J2 pad 2: /Power/B- -> unconnected-(J2-Pin_2-Pad2)
- J2 pad 3: /Power/B- -> unconnected-(J2-Pin_3-Pad3)
- J2 pad 4: /Power/B- -> unconnected-(J2-Pin_4-Pad4)
- J2 pad 43: /Networking/TX_CT -> /Networking/RX_CT
- J2 pad 44: /Networking/TX_CT -> /Networking/RX_CT
- J2 pad 45: /Networking/RX_CT -> /Networking/TX_CT
- J2 pad 46: /Networking/RX_CT -> /Networking/TX_CT
- J2 pad 47: /Networking/7_8 -> /Networking/4_5
- J2 pad 48: /Networking/7_8 -> /Networking/4_5
- J2 pad 49: /Networking/4_5 -> /Networking/7_8
- J2 pad 5: /Power/M1 -> unconnected-(J2-Pin_5-Pad5)
- J2 pad 50: /Networking/4_5 -> /Networking/7_8
- J2 pad 6: /Power/M0 -> unconnected-(J2-Pin_6-Pad6)
- J2 pad 7: /Power/M3 -> unconnected-(J2-Pin_7-Pad7)
- J2 pad 8: /Power/M2 -> unconnected-(J2-Pin_8-Pad8)
- J2 pad 9: /Power/B+ -> unconnected-(J2-Pin_9-Pad9)
- R1 pad 1: /I_SDA -> +3.3V
- R1 pad 2: +3.3V -> Net-(U1-VREG_AVDD)
- R2 pad 1: /I_SCL -> Net-(U1-XOUT)
- R2 pad 2: +3.3V -> Net-(C15-Pad2)
- T2 pad 2: Net-(T2-CT1) -> /Networking/TCT
- T2 pad 7: Net-(T2-CT2) -> /Networking/RCT
- TP78 pad 1: Net-(U4A-~{RESET}) -> Net-(U1-RUN)
- U4 pad 1: /NET_MISO -> Net-(U4-TXN)
- U4 pad 10: /Power_INT -> Net-(U4-EXRES1)
- U4 pad 11: /M_CLK -> +3.3V
- U4 pad 12: /M_MOSI -> unconnected-(U4-NC-Pad12)
- U4 pad 13: /F0_GPIO -> unconnected-(U4-NC-Pad13)
- U4 pad 14: /F1_GPIO -> GND
- U4 pad 15: /F2_GPIO -> +3.3V
- U4 pad 16: /F3_GPIO -> GND
- U4 pad 17: /F4_GPIO -> +3.3V
- U4 pad 18: /F5_GPIO -> unconnected-(U4-VBG-Pad18)
- U4 pad 19: /F6_GPIO -> GND
- U4 pad 2: /Power_CS -> Net-(U4-TXP)
- U4 pad 20: /F7_GPIO -> Net-(U4-TOCAP)
- U4 pad 21: /S0_GPIO -> +3.3V
- U4 pad 22: /S1_GPIO -> Net-(U4-1V2O)
- U4 pad 23: /S2_GPIO -> unconnected-(U4-RSVD-Pad23)
- U4 pad 24: /S3_GPIO -> Net-(D11-A)
- U4 pad 25: /S4_GPIO -> Net-(D12-A)
- U4 pad 26: /S5_GPIO -> Net-(D13-A)
- U4 pad 27: /S6_GPIO -> Net-(D14-A)
- U4 pad 28: /S7_GPIO -> +3.3V
- U4 pad 29: /SWDIO -> GND
- U4 pad 3: /NET_CLK -> GND
- U4 pad 30: /SWCLK -> Net-(U4-XI/CLKIN)
- U4 pad 31: GND -> Net-(U4-XO)
- U4 pad 32: unconnected-(U4A-VBAT-Pad32) -> /W5500_~{CS}
- U4 pad 33: unconnected-(U4A-5V-Pad33) -> /NET_CLK
- U4 pad 34: +3.3V -> /NET_MISO
- U4 pad 35: /USB_D- -> /NET_MOSI
- U4 pad 36: /USB_D+ -> /W5500_~{INT}
- U4 pad 37: unconnected-(U4A-SWDIO-Pad37) -> /W5500_~{RESET}
- U4 pad 39: Net-(U4A-~{RESET}) -> unconnected-(U4-RSVD-Pad39)
- U4 pad 4: /NET_MOSI -> +3.3V
- U4 pad 40: Net-(U4A-BOOTSEL) -> unconnected-(U4-RSVD-Pad40)
- U4 pad 41: /I_SDA -> unconnected-(U4-RSVD-Pad41)
- U4 pad 42: /I_SCL -> unconnected-(U4-RSVD-Pad42)
- U4 pad 43: /SD_CLK -> +3.3V
- U4 pad 44: /SD_CMD -> +3.3V
- U4 pad 45: /SD_D0 -> +3.3V
- U4 pad 46: /SD_D1 -> unconnected-(U4-NC-Pad46)
- U4 pad 47: /SD_D2 -> unconnected-(U4-NC-Pad47)
- U4 pad 48: /SD_D3 -> GND
- U4 pad 5: /CS0 -> Net-(U4-RXN)
- U4 pad 6: /CS1 -> Net-(U4-RXP)
- U4 pad 7: /CS2 -> unconnected-(U4-DNC-Pad7)
- U4 pad 8: /CS3 -> +3.3V
- U4 pad 9: /M_MISO -> GND
Routing:
- net +3.3V: track 327.7 -> 397.9 mm, vias 20 -> 28
- net /NET_MOSI: track 121.1 -> 186.0 mm
- net /NET_CLK: track 119.5 -> 183.4 mm
- net /~{PWR_RST}: track 124.6 -> 181.3 mm, vias 5 -> 7
- net +1V1: track 0.00 -> 54.3 mm
- net /Power/B+: track 53.0 -> 0.00 mm
- net /RAM_CS: track 0.00 -> 47.5 mm, vias 0 -> 2
- net /SWDIO: track 119.7 -> 162.6 mm, vias 2 -> 4
- net /NET_MISO: track 144.5 -> 186.9 mm, vias 4 -> 3
- net /Power_CS: track 70.8 -> 110.0 mm, vias 1 -> 2
- net Net-(U1-RUN): track 0.00 -> 38.8 mm, vias 0 -> 2
- net Net-(J4-Pin_1): track 0.00 -> 38.1 mm, vias 0 -> 2
- net /Power_INT: track 65.3 -> 102.7 mm
- net Net-(J4-Pin_2): track 0.00 -> 36.1 mm, vias 0 -> 2
- net /Power/M3: track 31.4 -> 0.00 mm
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Other:
- board text added: "GND"
- board text added: "SWCLK"
- board text added: "SWDIO"
- board text removed: "BOOTSEL"
- board text removed: "~{ACT}"
- board text removed: "~{LINK}"
- board text removed: "~{RST}"

Commit message: Finished PCBs
Parts:
- C14, C15: value 22pF -> 15pF
- L1: value 3.3uH -> AOTA-B201610S3R3-101-T; footprint Inductor_SMD:L_Pulse_PA4340 -> Snapeda:0806
- Y1: value Crystal_GND24 -> ABM8-272-T3
- Y2: value 25MHZ -> ABM3C-25.000MHZ-D4Y-T
- moved C13 6.49 mm to (191.5, 130.4)
- moved L1 2.83 mm to (189.9, 128.8)
- moved C3 1.08 mm to (192.7, 131.7)
Routing:
- net +1V1: track 54.3 -> 50.0 mm
- net Net-(U1-VREG_LX): track 9.28 -> 6.40 mm
- net GND: track 18.9 -> 21.4 mm
- net +3.3V: track 397.9 -> 396.6 mm, vias 28 -> 27

Commit message: Started code, commiting before adding submodules
Parts:
- moved C4 1.02 mm to (201.2, 132.7)
Connections:
- J6 pad 13: GND -> /CS_~{EN}
- J6 pad 14: /S7_GPIO -> GND
- J6 pad 15: /S6_GPIO -> /S7_GPIO
- J6 pad 16: /S5_GPIO -> /S6_GPIO
- J6 pad 17: /S4_GPIO -> /S5_GPIO
- J6 pad 18: /S3_GPIO -> /S4_GPIO
- J6 pad 19: /S2_GPIO -> /S3_GPIO
- J6 pad 20: /S1_GPIO -> /S2_GPIO
- J6 pad 21: /S0_GPIO -> /S1_GPIO
- J6 pad 22: /F7_GPIO -> /S0_GPIO
- J6 pad 23: /F6_GPIO -> /F7_GPIO
- J6 pad 24: /F5_GPIO -> /F6_GPIO
- J6 pad 25: /F4_GPIO -> /F5_GPIO
- J6 pad 26: /F3_GPIO -> /F4_GPIO
- J6 pad 27: /F2_GPIO -> /F3_GPIO
- J6 pad 28: /F1_GPIO -> /F2_GPIO
- J6 pad 29: /F0_GPIO -> /F1_GPIO
- J6 pad 30: GND -> /F0_GPIO
- J6 pad 31: +3.3V -> GND
- J6 pad 34: GND -> +3.3V
- J6 pad 36: VCC -> GND
- U1 pad 49: unconnected-(U1-GPIO40/ADC0-Pad49) -> /CS_~{EN}
Routing:
- net /CS_~{EN}: track 0.00 -> 38.1 mm, vias 0 -> 2
- net /S4_GPIO: track 18.8 -> 22.7 mm
- net /F2_GPIO: track 20.2 -> 24.0 mm
- net /F4_GPIO: track 18.7 -> 22.4 mm
- net /S0_GPIO: track 16.1 -> 19.7 mm
- net /S7_GPIO: track 24.0 -> 20.4 mm
- net /F6_GPIO: track 17.4 -> 21.0 mm
- net /S2_GPIO: track 16.5 -> 20.0 mm
- net /S5_GPIO: track 22.6 -> 19.6 mm
- net /F1_GPIO: track 24.7 -> 21.6 mm
- net /F0_GPIO: track 22.4 -> 25.3 mm
- net /S3_GPIO: track 19.5 -> 17.0 mm
- net /S6_GPIO: track 20.3 -> 22.8 mm
- net /F3_GPIO: track 22.7 -> 20.2 mm
- net /S1_GPIO: track 19.5 -> 17.0 mm
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