File: PCB/Virgil Controller/Virgil Controller.kicad_sch (KiCad schematic)
At the start: 12 parts, among them J1 USB_C_Receptacle_USB2.0_16P, J3 503398-1892, J6 SBH11-PBPC-D25-RA-BK, U4 RP2350_Stamp_XL

Commit message: Created actually good readme
Parts:
- removed TP77: BootSel, Connector_PinHeader_2.00mm:PinHeader_1x01_P2.00mm_Vertical, symbol Connector:TestPoint
- removed U4: RP2350_Stamp_XL, Snapeda:RP2xxx_Stamp_XL_FlexyPin, symbol RP2xxx_Stamp:RP2350_Stamp_XL
- added C1, C13: 4.7uF, Capacitor_SMD:C_0805_2012Metric, symbol Device:C
- added C10, C11, C12, C2, C3, C4, C5, C6, C7, C8, C9: .1uF, Capacitor_SMD:C_0603_1608Metric, symbol Device:C
- added C14, C15: 22pF, Capacitor_SMD:C_0603_1608Metric, symbol Device:C
- added J4: Conn_01x03_Pin, Connector_PinSocket_2.54mm:PinSocket_1x03_P2.54mm_Vertical, symbol Connector:Conn_01x03_Pin
- added L1: 3.3uH, Inductor_SMD:L_Pulse_PA4340, symbol Device:L
- added R20, R21: 27Ω, Resistor_SMD:R_0603_1608Metric, symbol Device:R_US
- added R4, R5: 4.7Ω, Resistor_SMD:R_0805_2012Metric, symbol Device:R_US
- added U1: RP2350B, Package_DFN_QFN:QFN-80-1EP_10x10mm_P0.4mm_EP3.4x3.4mm, symbol MCU_RaspberryPi:RP2350B
- added U2, U3: W25Q16JVSS, Package_SO:SOIC-8_5.3x5.3mm_P1.27mm, symbol Memory_Flash:W25Q16JVSS
- added Y1: Crystal_GND24, Crystal:Crystal_SMD_Abracon_ABM8G-4Pin_3.2x2.5mm, symbol Device:Crystal_GND24
- R1: value 4.7Ω -> 33Ω; footprint Resistor_SMD:R_0805_2012Metric -> Resistor_SMD:R_0603_1608Metric
- R2: value 4.7Ω -> 1kΩ; footprint Resistor_SMD:R_0805_2012Metric -> Resistor_SMD:R_0603_1608Metric
Connections:
- net +3.3V: now also R1.1, C10.1, C2.1, C3.1, C4.1, C5.1, C6.1, C7.1, C8.1, C9.1, R4.2, R5.2, U1.15 (IOVDD), U1.24 (IOVDD), U1.29 (IOVDD), U1.41 (IOVDD), U1.5 (IOVDD), U1.50 (IOVDD), U1.59 (ADC_AVDD), U1.60 (IOVDD), U1.64 (VREG_VIN), U1.69 (QSPI_IOVDD), U1.76 (IOVDD), U2.8 (VCC), U3.8 (VCC); no longer R1.2, R2.2
- net CS0: now also U1.1 (GPIO4)
- net CS1: now also U1.2 (GPIO5)
- net CS2: now also U1.3 (GPIO6)
- net CS3: now also U1.4 (GPIO7)
- net F0_GPIO: now also U1.11 (GPIO12)
- net F1_GPIO: now also U1.12 (GPIO13)
- net F2_GPIO: now also U1.13 (GPIO14)
- net F3_GPIO: now also U1.14 (GPIO15)
- net F4_GPIO: now also U1.16 (GPIO16)
- net F5_GPIO: now also U1.17 (GPIO17)
- net F6_GPIO: now also U1.18 (GPIO18)
- net F7_GPIO: now also U1.19 (GPIO19)
- net GND: now also C1.1, C10.2, C11.2, C12.2, C13.2, C14.1, C15.1, C2.2, C3.2, C4.2, C5.2, C6.2, C7.2, C8.2, C9.2, J4.3 (Pin_3), U1.62 (VREG_PGND), U1.81 (GND), U2.4 (GND), U3.4 (GND), Y1.2 (G), Y1.4 (G)
- net I_SCL: now also R5.1, U1.39 (GPIO31); no longer R2.1
- net I_SDA: now also R4.1, U1.38 (GPIO30); no longer R1.1
- net M_CLK: now also U1.8 (GPIO10)
- net M_MISO: now also U1.6 (GPIO8)
- net M_MOSI: now also U1.9 (GPIO11)
- net NET_CLK: now also U1.79 (GPIO2)
- net NET_MISO: now also U1.77 (GPIO0)
- net NET_MOSI: now also U1.80 (GPIO3)
- net Power_CS: now also U1.78 (GPIO1)
- net Power_INT: now also U1.7 (GPIO9)
- net RADIO_CS: now also U1.53 (GPIO42/ADC2)
- net RADIO_EN: now also U1.55 (GPIO44/ADC4)
- net RADIO_~{INT}: now also U1.54 (GPIO43/ADC3)
- net S0_GPIO: now also U1.20 (GPIO20)
- net S1_GPIO: now also U1.21 (GPIO21)
- net S2_GPIO: now also U1.22 (GPIO22)
- net S3_GPIO: now also U1.23 (GPIO23)
- net S4_GPIO: now also U1.25 (GPIO24)
- net S5_GPIO: now also U1.26 (GPIO25)
- net S6_GPIO: now also U1.27 (GPIO26)
- net S7_GPIO: now also U1.28 (GPIO27)
- net SD_CLK: now also U1.40 (GPIO32)
- net SD_CMD: now also U1.42 (GPIO33)
- net SD_D0: now also U1.43 (GPIO34)
- net SD_D1: now also U1.44 (GPIO35)
- net SD_D2: now also U1.45 (GPIO36)
- net SD_D3: now also U1.46 (GPIO37)
- net SD_DET: now also U1.47 (GPIO38)
- net SWCLK: now also U1.37 (GPIO29)
- net SWDIO: now also U1.36 (GPIO28)
- net USB_D+: now also R21.1
- net USB_D-: now also R20.1
- net W5500_~{CS}: now also U1.56 (GPIO45/ADC5)
- net W5500_~{INT}: now also U1.57 (GPIO46/ADC6)
- net W5500_~{RESET}: now also U1.58 (GPIO47/ADC7)
- net ~{PWR_RST}: now also U1.48 (GPIO39)
- net at TP78.1: now also U1.35 (RUN)
- new net: C1.2, R1.2, U1.61 (VREG_AVDD)
- new net: R2.1, U1.31 (XOUT)
- new net: C15.2, R2.2, Y1.3
- new net: R21.2, U1.67 (USB_DP)
- new net: C14.2, U1.30 (XIN), Y1.1
- new net: U1.75 (~{QSPI_SS}), U2.1 (~{CS})
- new net: R20.2, U1.66 (USB_DM)
- new net: J4.1 (Pin_1), U1.33 (SWCLK)
- new net: J4.2 (Pin_2), U1.34 (SWDIO)
- new net: L1.1, U1.63 (VREG_LX)
- new net +1V1: C11.1, C12.1, C13.1, L1.2, U1.10 (DVDD), U1.32 (DVDD), U1.51 (DVDD), U1.65 (VREG_FB)
- new net QSPI_SCLK: U1.71 (QSPI_SCLK), U2.6 (CLK), U3.6 (CLK)
- new net QSPI_SD0: U1.72 (QSPI_SD0), U2.5 (DI/IO_{0}), U3.5 (DI/IO_{0})
- new net QSPI_SD1: U1.74 (QSPI_SD1), U2.2 (DO/IO_{1}), U3.2 (DO/IO_{1})
- new net QSPI_SD2: U1.73 (QSPI_SD2), U2.3 (~{WP}/IO_{2}), U3.3 (~{WP}/IO_{2})
- new net QSPI_SD3: U1.70 (QSPI_SD3), U2.7 (~{HOLD}/~{RESET}/IO_{3}), U3.7 (~{HOLD}/~{RESET}/IO_{3})
- new net RAM_CS: U1.52 (GPIO41/ADC1), U3.1 (~{CS})
- no-connect marks 8 -> 3
Other:
- moved on the sheet: H1, H2, H3, H4

Commit message: Finished PCBs
Parts:
- C14, C15: value 22pF -> 15pF
- L1: value 3.3uH -> AOTA-B201610S3R3-101-T; footprint Inductor_SMD:L_Pulse_PA4340 -> Snapeda:0806
- Y1: value Crystal_GND24 -> ABM8-272-T3
Changed lines of the file:
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@@
 			)
 		)
-		(property "Value" "22pF"
+		(property "Value" "15pF"
 			(at 130.81 129.5399 0)
 			(show_name no)
@@
 		(fields_autoplaced yes)
 		(property "Reference" "Y1"
-			(at 141.605 116.205 0)
+			(at 141.605 115.57 0)
 			(show_name no)
 			(do_not_autoplace no)
@@
 			)
 		)
-		(property "Value" "Crystal_GND24"
-			(at 141.605 118.745 0)
+		(property "Value" "ABM8-272-T3"
+			(at 141.605 118.11 0)
 			(show_name no)
 			(do_not_autoplace no)
@@
 			)
 		)
-		(property "Value" "22pF"
+		(property "Value" "15pF"
 			(at 152.4 129.5399 0)
 			(show_name no)
@@
 			)
 		)
-		(property "Value" "3.3uH"
+		(property "Value" "AOTA-B201610S3R3-101-T"
 			(at 193.04 30.48 90)
 			(show_name no)
@@
 			)
 		)
-		(property "Footprint" "Inductor_SMD:L_Pulse_PA4340"
+		(property "Footprint" "Snapeda:0806"
 			(at 193.04 33.02 0)
 			(hide yes)

Commit message: Started code, commiting before adding submodules
Connections:
- net +3.3V: now also J6.34 (Pin_34); no longer J6.31 (Pin_31)
- net F0_GPIO: now also J6.30 (Pin_30); no longer J6.29 (Pin_29)
- net F1_GPIO: now also J6.29 (Pin_29); no longer J6.28 (Pin_28)
- net F2_GPIO: now also J6.28 (Pin_28); no longer J6.27 (Pin_27)
- net F3_GPIO: now also J6.27 (Pin_27); no longer J6.26 (Pin_26)
- net F4_GPIO: now also J6.26 (Pin_26); no longer J6.25 (Pin_25)
- net F5_GPIO: now also J6.25 (Pin_25); no longer J6.24 (Pin_24)
- net F6_GPIO: now also J6.24 (Pin_24); no longer J6.23 (Pin_23)
- net F7_GPIO: now also J6.23 (Pin_23); no longer J6.22 (Pin_22)
- net GND: now also J6.14 (Pin_14), J6.31 (Pin_31), J6.36 (Pin_36); no longer J6.13 (Pin_13), J6.30 (Pin_30), J6.34 (Pin_34)
- net S0_GPIO: now also J6.22 (Pin_22); no longer J6.21 (Pin_21)
- net S1_GPIO: now also J6.21 (Pin_21); no longer J6.20 (Pin_20)
- net S2_GPIO: now also J6.20 (Pin_20); no longer J6.19 (Pin_19)
- net S3_GPIO: now also J6.19 (Pin_19); no longer J6.18 (Pin_18)
- net S4_GPIO: now also J6.18 (Pin_18); no longer J6.17 (Pin_17)
- net S5_GPIO: now also J6.17 (Pin_17); no longer J6.16 (Pin_16)
- net S6_GPIO: now also J6.16 (Pin_16); no longer J6.15 (Pin_15)
- net S7_GPIO: now also J6.15 (Pin_15); no longer J6.14 (Pin_14)
- net VCC: no longer J6.36 (Pin_36)
- net CS_~{EN}: now reaches U1.49 (GPIO40/ADC0)
- net CS_~{EN}: now also J6.13 (Pin_13)
