File: PCB/Virgil Power/Monitoring.kicad_sch (KiCad schematic)
At the start: 11 parts, among them U10 INA226, U12 INA226, U13 BTS50080-1TEA, U3 INA226, U6 XIAO-RP2040-SMD, U8 INA226

Commit message: Created actually good readme
Changed lines of the file:
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@@
 		(fields_autoplaced yes)
 		(property "Reference" "U13"
-			(at 80.645 65.405 0)
+			(at 80.645 64.77 0)
 			(effects
 				(font
@@
 		)
 		(property "Value" "BTS50080-1TEA"
-			(at 80.645 67.945 0)
+			(at 80.645 67.31 0)
 			(effects
 				(font
