File: PCB/Virgil Power/Virgil Power.kicad_pcb (KiCad board)
At the start: 2 copper layers, 89 x 113 mm, 71 parts, among them J2 Barrel_Jack_MountingPin, J3 Conn_02x25_Odd_Even, U1 TPS563300, U10 INA226, U11 LTV-356T, U12 INA226, U13 BTS50080-1TEA, U2 TPS563300, U3 INA226, U4 TPS563300, U5 AG59612-LPB, U6 XIAO-RP2040-SMD, U7 MCP4562T-503E/MF, U8 INA226, U9 LTV-356T

Commit message: Created actually good readme
Parts:
- moved J2 49.8 mm to (135.0, 48.0), turned to -90 degrees
- moved U11 12.2 mm to (148.0, 85.0)
- moved U9 12.2 mm to (153.0, 85.0)
- moved U5 10.4 mm to (151.0, 65.0)
- moved D3 6.16 mm to (175.0, 59.4)
- moved D4 6.16 mm to (180.0, 59.4)
- moved D6 6.16 mm to (185.0, 59.4)
- moved D8 6.16 mm to (190.0, 59.4)
- moved D1 6.16 mm to (175.0, 76.3)
- moved D2 6.16 mm to (180.0, 76.3)
- moved D5 6.16 mm to (185.0, 76.3)
- moved D7 6.16 mm to (190.0, 76.3)
Routing:
- net /Monitoring/POE+: track 97.3 -> 90.1 mm
- net /Monitoring/POE++: track 92.1 -> 84.9 mm
- net Net-(U5-TYP3-DET): track 30.6 -> 35.1 mm
- net Net-(U5-TYP2-DET): track 29.5 -> 34.0 mm, vias 2 -> 0
- net /POE/PD-: track 22.9 -> 27.0 mm
- net /Monitoring/~{MOT_EN}: track 123.8 -> 121.5 mm
- net /POE_0: track 39.3 -> 37.2 mm
- net /POE_1: track 32.7 -> 31.1 mm
- net /POE_2: track 26.5 -> 25.1 mm
- net /POE/PD+: track 45.0 -> 45.8 mm
