File: PCB/Ribbon Adaptor/Ribbon Adaptor.kicad_sch (KiCad schematic)
At the start: 7 parts, among them J1 10056847-101LF, J2 SFV20R-2STE1HLF, J3 SFV20R-2STE1HLF

Commit message: Finished PCBs
Parts:
- removed J3: SFV20R-2STE1HLF, Snapeda:AMPHENOL_SFV20R-2STE1HLF, symbol Snapeda:SFV20R-2STE1HLF
- J1: now not fitted
- J2: value SFV20R-2STE1HLF -> AFC07-S20FCC-00

Commit message: Started code, commiting before adding submodules
Parts:
- J2: footprint Snapeda:AMPHENOL_SFV20R-2STE1HLF -> Snapeda:JUSHUO AFC07-S20FCC-00
Changed lines of the file:
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@@
 			)
 		)
-		(property "Footprint" "Snapeda:AMPHENOL_SFV20R-2STE1HLF"
+		(property "Footprint" "Snapeda:JUSHUO AFC07-S20FCC-00"
 			(at 121.285 71.755 0)
 			(hide yes)
