File: PCB/Virgil Backplane/Virgil Backplane.kicad_pcb (KiCad board)
At the start: 4 copper layers, 212 x 46 mm, 38 parts, among them J1 SBH11-PBPC-D25-RA-BK, J10 10056847-101LF, J11 10056847-101LF, J12 10056847-101LF, J13 10056847-101LF, J14 10056847-101LF, J15 10056847-101LF, J16 10056847-101LF, J17 10056847-101LF, J2 10056847-101LF, J3 10056847-101LF, J4 10056847-101LF, J5 10056847-101LF, J6 10056847-101LF, J7 10056847-101LF, J8 10056847-101LF, J9 10056847-101LF, U1 MCP23017T-E/SS, U2 MCP23017T-E/SS, U20 SN74CBTLV1G125DCKR, U21 SN74CBTLV1G125DCKR, U22 SN74CBTLV1G125DCKR, U23 SN74CBTLV1G125DCKR, U24 SN74CBTLV1G125DCKR, U25 SN74CBTLV1G125DCKR, U26 SN74CBTLV1G125DCKR, U27 SN74CBTLV1G125DCKR, U28 SN74CBTLV1G125DCKR, U29 SN74CBTLV1G125DCKR, U30 SN74CBTLV1G125DCKR, U31 SN74CBTLV1G125DCKR, U32 SN74CBTLV1G125DCKR, U33 SN74CBTLV1G125DCKR, U34 SN74CBTLV1G125DCKR, U35 SN74CBTLV1G125DCKR, U5 CD74HC154M96

Commit message: Started code, commiting before adding submodules
Connections:
- J1 pad 13: GND -> /CS_~{EN}
- J1 pad 14: /S7_GPIO -> GND
- J1 pad 15: /S6_GPIO -> /S7_GPIO
- J1 pad 16: /S5_GPIO -> /S6_GPIO
- J1 pad 17: /S4_GPIO -> /S5_GPIO
- J1 pad 18: /S3_GPIO -> /S4_GPIO
- J1 pad 19: /S2_GPIO -> /S3_GPIO
- J1 pad 20: /S1_GPIO -> /S2_GPIO
- J1 pad 21: /S0_GPIO -> /S1_GPIO
- J1 pad 22: /F7_GPIO -> /S0_GPIO
- J1 pad 23: /F6_GPIO -> /F7_GPIO
- J1 pad 24: /F5_GPIO -> /F6_GPIO
- J1 pad 25: /F4_GPIO -> /F5_GPIO
- J1 pad 26: /F3_GPIO -> /F4_GPIO
- J1 pad 27: /F2_GPIO -> /F3_GPIO
- J1 pad 28: /F1_GPIO -> /F2_GPIO
- J1 pad 29: /F0_GPIO -> /F1_GPIO
- J1 pad 30: GND -> /F0_GPIO
- J1 pad 31: +3.3V -> GND
- J1 pad 34: GND -> +3.3V
- J1 pad 36: VCC -> GND
- U5 pad 18: GND -> /CS_~{EN}
- U5 pad 19: GND -> /CS_~{EN}
Routing:
- net /CS_~{EN}: track 0.00 -> 130.9 mm, vias 0 -> 2
- net /F3_GPIO: track 76.1 -> 72.5 mm
- net /F5_GPIO: track 21.2 -> 17.6 mm
- net /S7_GPIO: track 45.2 -> 48.8 mm
- net /S2_GPIO: track 109.7 -> 106.1 mm
- net /F6_GPIO: track 23.6 -> 27.2 mm
- net /F0_GPIO: track 155.3 -> 158.9 mm
- net /S4_GPIO: track 54.7 -> 51.2 mm
- net /F1_GPIO: track 131.1 -> 127.8 mm
- net /S0_GPIO: track 164.6 -> 161.4 mm
- net /S1_GPIO: track 134.1 -> 136.6 mm
- net /F7_GPIO: track 54.2 -> 51.6 mm
- net /S5_GPIO: track 24.3 -> 26.8 mm
- net /F2_GPIO: track 100.6 -> 103.1 mm
- net /S6_GPIO: track 21.0 -> 18.4 mm
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