File: PCB/Virgil Backplane/Virgil Backplane.kicad_sch (KiCad schematic)
At the start: 8 parts, among them J1 SBH11-PBPC-D25-RA-BK, U1 MCP23017T-E/SS, U2 MCP23017T-E/SS, U5 CD74HC154M96

Commit message: Started code, commiting before adding submodules
Connections:
- net +3.3V: now also J1.34 (Pin_34); no longer J1.31 (Pin_31)
- net F0_GPIO: now also J1.30 (Pin_30); no longer J1.29 (Pin_29)
- net F1_GPIO: now also J1.29 (Pin_29); no longer J1.28 (Pin_28)
- net F2_GPIO: now also J1.28 (Pin_28); no longer J1.27 (Pin_27)
- net F3_GPIO: now also J1.27 (Pin_27); no longer J1.26 (Pin_26)
- net F4_GPIO: now also J1.26 (Pin_26); no longer J1.25 (Pin_25)
- net F5_GPIO: now also J1.25 (Pin_25); no longer J1.24 (Pin_24)
- net F6_GPIO: now also J1.24 (Pin_24); no longer J1.23 (Pin_23)
- net F7_GPIO: now also J1.23 (Pin_23); no longer J1.22 (Pin_22)
- net GND: now also J1.14 (Pin_14), J1.31 (Pin_31), J1.36 (Pin_36); no longer J1.13 (Pin_13), J1.30 (Pin_30), J1.34 (Pin_34), U5.18 (*E1), U5.19 (*E2)
- net S0_GPIO: now also J1.22 (Pin_22); no longer J1.21 (Pin_21)
- net S1_GPIO: now also J1.21 (Pin_21); no longer J1.20 (Pin_20)
- net S2_GPIO: now also J1.20 (Pin_20); no longer J1.19 (Pin_19)
- net S3_GPIO: now also J1.19 (Pin_19); no longer J1.18 (Pin_18)
- net S4_GPIO: now also J1.18 (Pin_18); no longer J1.17 (Pin_17)
- net S5_GPIO: now also J1.17 (Pin_17); no longer J1.16 (Pin_16)
- net S6_GPIO: now also J1.16 (Pin_16); no longer J1.15 (Pin_15)
- net S7_GPIO: now also J1.15 (Pin_15); no longer J1.14 (Pin_14)
- net VCC: no longer J1.36 (Pin_36)
- new net CS_~{EN}: J1.13 (Pin_13), U5.18 (*E1), U5.19 (*E2)
